File: hardware/r1.3/mmdvm_hs_dual_hat.sch (KiCad schematic (older format))
At the start: 70 parts, among them P1 SMA, P2 SMA, U1 ADF7021, U2 ADF7021, X1 TCXO

Commit message: Cleaned up libraries and schematics
Preparation for Revision 2.0
Parts:
- X1: symbol mmdvm_hs_dual_hat-rescue:TCXO_DFAS11-RESCUE-mmdvm_hs_dual_hat-mmdvm_hs_dual_hat-rescue -> Oscillator:ABLNO
Connections:
- net +3V3: now also X1.2 (GND); no longer X1.4 (VCC)
- net GND: now also X1.4 (VDD); no longer X1.2 (GND)
Other:
- moved on the sheet: C42
Changed lines of the file:
@@
 EESchema Schematic File Version 4
-LIBS:mmdvm_hs_dual_hat-cache
-EELAYER 26 0
+EELAYER 30 0
 EELAYER END
 $Descr A4 11693 8268
@@
 $EndComp
 $Comp
-L mmdvm_hs_dual_hat-rescue:TCXO_DFAS11-RESCUE-mmdvm_hs_dual_hat-mmdvm_hs_dual_hat-rescue X1
+L Oscillator:ABLNO X1
 U 1 1 5897A831
-P 6250 1300
-F 0 "X1" H 6250 1600 50  0000 C CNN
-F 1 "TCXO" H 6250 1300 50  0000 C CNN
-F 2 "Crystals:Crystal_SMD_3225-4pin_3.2x2.5mm" H 6250 1300 50  0001 C CNN
-F 3 "http://www.mouser.com/ds/2/122/ECS-TXO-3225-608196.pdf" H 6250 1300 50  0001 C CNN
-F 4 "ECS" H -800 -3200 50  0001 C CNN "MFR"
-F 5 "ECS-TXO-3225-147.4-TR" H -800 -3200 50  0001 C CNN "MPN"
-F 6 "Mouser" H -800 -3200 50  0001 C CNN "SPR"
-F 7 "520-TXO-3225-14.74T" H -800 -3200 50  0001 C CNN "SPN"
-F 8 "" H -800 -3200 50  0001 C CNN "SPURL"
-	1    6250 1300
+P 6250 1200
+F 0 "X1" H 6250 1500 50  0000 C CNN
+F 1 "TCXO" H 6250 1200 50  0000 C CNN
+F 2 "Crystals:Crystal_SMD_3225-4pin_3.2x2.5mm" H 6250 1200 50  0001 C CNN
+F 3 "http://www.mouser.com/ds/2/122/ECS-TXO-3225-608196.pdf" H 6250 1200 50  0001 C CNN
+F 4 "ECS" H -800 -3300 50  0001 C CNN "MFR"
+F 5 "ECS-TXO-3225-147.4-TR" H -800 -3300 50  0001 C CNN "MPN"
+F 6 "Mouser" H -800 -3300 50  0001 C CNN "SPR"
+F 7 "520-TXO-3225-14.74T" H -800 -3300 50  0001 C CNN "SPN"
+F 8 "" H -800 -3300 50  0001 C CNN "SPURL"
+	1    6250 1200
 	-1   0    0    1
 $EndComp
@@
 L power:GND #PWR069
 U 1 1 5897AC36
-P 5400 1150
-F 0 "#PWR069" H 5400 900 50  0001 C CNN
-F 1 "GND" H 5400 1000 50  0000 C CNN
-F 2 "" H 5400 1150 50  0000 C CNN
-F 3 "" H 5400 1150 50  0000 C CNN
-	1    5400 1150
-	0    1    1    0
+P 6250 1650
+F 0 "#PWR069" H 6250 1400 50  0001 C CNN
+F 1 "GND" H 6250 1500 50  0000 C CNN
+F 2 "" H 6250 1650 50  0000 C CNN
+F 3 "" H 6250 1650 50  0000 C CNN
+	1    6250 1650
+	1    0    0    -1
 $EndComp
 $Comp
 L power:GND #PWR075
 U 1 1 5897AF7A
-P 7100 1850
-F 0 "#PWR075" H 7100 1600 50  0001 C CNN
-F 1 "GND" H 7100 1700 50  0000 C CNN
-F 2 "" H 7100 1850 50  0000 C CNN
-F 3 "" H 7100 1850 50  0000 C CNN
-	1    7100 1850
+P 6900 1200
+F 0 "#PWR075" H 6900 950 50  0001 C CNN
+F 1 "GND" H 6900 1050 50  0000 C CNN
+F 2 "" H 6900 1200 50  0000 C CNN
+F 3 "" H 6900 1200 50  0000 C CNN
+	1    6900 1200
 	1    0    0    -1
 $EndComp
@@
 L mmdvm_hs_dual_hat-rescue:C-device-mmdvm_hs_dual_hat-rescue C42
 U 1 1 5897B23C
-P 7100 1650
-F 0 "C42" H 7125 1750 50  0000 L CNN
-F 1 "10n" H 7125 1550 50  0000 L CNN
-F 2 "Capacitors_SMD:C_0402" H 7138 1500 50  0001 C CNN
-F 3 "https://www.mouser.com/ds/2/427/vjw1bcbascomseries-223529.pdf" H 7100 1650 50  0001 C CNN
-F 4 "Vishay / Vitramon" H 1050 -2900 50  0001 C CNN "MFR"
-F 5 "VJ0402Y103KXJCW1BC" H 1050 -2900 50  0001 C CNN "MPN"
-F 6 "Mouser" H 1050 -2900 50  0001 C CNN "SPR"
-F 7 "77-VJ0402Y103KXJCBC" H 1050 -2900 50  0001 C CNN "SPN"
-F 8 "" H 1050 -2900 50  0001 C CNN "SPURL"
-	1    7100 1650
+P 6900 1000
+F 0 "C42" H 6925 1100 50  0000 L CNN
+F 1 "10n" H 6925 900 50  0000 L CNN
+F 2 "Capacitors_SMD:C_0402" H 6938 850 50  0001 C CNN
+F 3 "https://www.mouser.com/ds/2/427/vjw1bcbascomseries-223529.pdf" H 6900 1000 50  0001 C CNN
+F 4 "Vishay / Vitramon" H 850 -3550 50  0001 C CNN "MFR"
+F 5 "VJ0402Y103KXJCW1BC" H 850 -3550 50  0001 C CNN "MPN"
+F 6 "Mouser" H 850 -3550 50  0001 C CNN "SPR"
+F 7 "77-VJ0402Y103KXJCBC" H 850 -3550 50  0001 C CNN "SPN"
+F 8 "" H 850 -3550 50  0001 C CNN "SPURL"
+	1    6900 1000
 	1    0    0    -1
 $EndComp
@@
 L power:+3.3V #PWR074
 U 1 1 5A6B3FE9
-P 7100 1350
-F 0 "#PWR074" H 7100 1200 50  0001 C CNN
-F 1 "+3.3V" H 7100 1490 50  0000 C CNN
-F 2 "" H 7100 1350 50  0000 C CNN
-F 3 "" H 7100 1350 50  0000 C CNN
-	1    7100 1350
+P 6900 700
+F 0 "#PWR074" H 6900 550 50  0001 C CNN
+F 1 "+3.3V" H 6900 840 50  0000 C CNN
+F 2 "" H 6900 700 50  0000 C CNN
+F 3 "" H 6900 700 50  0000 C CNN
+	1    6900 700
 	1    0    0    -1
 $EndComp
@@
 F 0 "W1" H 1608 5015 50  0000 L CNN
 F 1 "TEST_1P" H 1608 4924 50  0000 L CNN
-F 2 "Connectors_TestPoints:Test_Point_Pad_1.0x1.0mm" H 1608 4833 50  0000 L CNN
+F 2 "Connectors_TestPoints:Test_Point_Pad_1.0x1.0mm" H 1608 4833 50  0001 L CNN
 F 3 "" H 1750 4850 50  0000 C CNN
 F 4 "" H 0   0   50  0001 C CNN "MFR"
@@
 F 0 "W2" H 1608 4665 50  0000 L CNN
 F 1 "TEST_1P" H 1608 4574 50  0000 L CNN
-F 2 "Connectors_TestPoints:Test_Point_Pad_1.0x1.0mm" H 1608 4483 50  0000 L CNN
+F 2 "Connectors_TestPoints:Test_Point_Pad_1.0x1.0mm" H 1608 4483 50  0001 L CNN
 F 3 "" H 1750 4500 50  0000 C CNN
 F 4 "" H 0   0   50  0001 C CNN "MFR"
@@
 	4250 4950 4250 4850
 Wire Wire Line
-	7100 1350 7100 1450
-Wire Wire Line
-	7100 1800 7100 1850
+	6900 700  6900 800
+Wire Wire Line
+	6900 1150 6900 1200
 Wire Wire Line
 	850  2750 950  2750
@@
 	4450 5250 4450 5350
 Wire Wire Line
-	6950 1450 7100 1450
-Wire Wire Line
 	3150 4400 3150 4350
 Wire Wire Line
@@
 	1900 6250 3000 6250
 Wire Wire Line
-	7100 1450 7100 1500
+	6900 800  6900 850
 Wire Wire Line
 	2850 5300 3050 5300
@@
 	5250 1450 5450 1450
 Wire Wire Line
-	5400 1150 5550 1150
+	6250 1650 6250 1500
 Wire Wire Line
 	5450 1450 5450 1900
@@
 Connection ~ 1150 2650
 Connection ~ 1100 6450
-Connection ~ 7100 1450
+Connection ~ 6900 800
 Connection ~ 5450 1450
 Connection ~ 1700 1800
@@
 NoConn ~ 4550 5350
 NoConn ~ 4650 5350
-NoConn ~ 6950 1150
+NoConn ~ 6650 1200
 NoConn ~ 5200 2750
 NoConn ~ 4600 3800
@@
 NoConn ~ 5200 2150
 NoConn ~ 5150 5950
+Wire Wire Line
+	6250 800  6250 900
+Wire Wire Line
+	6250 800  6900 800
+Wire Wire Line
+	5850 1200 5550 1200
+Wire Wire Line
+	5550 1200 5550 1450
 $EndSCHEMATC
